File: eacs_hardware/eacs_hardware.kicad_sch (KiCad schematic)
At the start: 34 parts, among them J1 IEC_60320_C14_Receptacle, Q1 S8050, Q2 SS8050, Q3 SS8050, Q4 SS8050, Q5 SS8050, SW1 SW_Push, T1 6:1, U1 ESP32-WROOM-32

Commit message: Completed schematics
Other:
- note added: "0.1"
- note added: "23 December 2024"
Changed lines of the file:
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@@
+		)
+	)
+	(text "0.1"
+		(exclude_from_sim no)
+		(at 271.018 193.548 0)
+		(effects
+			(font
+				(face "3270 Nerd Font")
+				(size 2.032 2.032)
+				(thickness 0.254)
+				(bold yes)
+				(color 0 0 0 1)
+			)
 		)
 	)
@@
 				(thickness 0.254)
 				(bold yes)
+				(color 0 0 0 1)
+			)
+		)
+	)
+	(text "23 December 2024\n"
+		(exclude_from_sim no)
+		(at 216.408 193.802 0)
+		(effects
+			(font
+				(face "3270 Nerd Font")
+				(size 2.032 2.032)
+				(thickness 0.254)
+				(bold yes)
